File: electric/scheme/cam-chassis.sch (KiCad schematic (older format))
At the start: 48 parts, among them IC1 ATMEGA8-AI, K1 pyro, P1 TST, P2 TST, P3 TST, P4 TST, P5 TST, P6 TST, P7 servo, Q3 bc857, Q4 bc847, Q5 irlml2244, Q6 NPN, Q7 irlml2244, U1 crystal-4pin, U2 MICRO-USB-B

Commit message: a
Parts:
- removed U2: MICRO-USB-B, micro-usb-b:micro-usb-b, symbol MICRO-USB-B
- added U?: MINI-USB-B, symbol MINI-USB-B
Connections:
- wire segments 145 -> 134
Changed lines of the file:
@@
 LIBS:memory
 LIBS:xilinx
-LIBS:special
 LIBS:microcontrollers
 LIBS:dsp
@@
 d+
 $Comp
-L MICRO-USB-B U2
-U 1 1 55219FEF
-P 10400 5950
-F 0 "U2" H 10400 5350 60  0000 C CNN
-F 1 "MICRO-USB-B" H 10400 5800 60  0000 C CNN
-F 2 "micro-usb-b:micro-usb-b" H 10400 5950 60  0000 C CNN
-F 3 "~" H 10400 5950 60  0000 C CNN
-	1    10400 5950
-	0    -1   1    0
-$EndComp
-$Comp
 L R R16
 U 1 1 5521A06E
@@
 F 3 "" H 9150 6800 60  0000 C CNN
 	1    9150 6800
-	1    0    0    -1
-$EndComp
-$Comp
-L GND #PWR016
-U 1 1 5521A48D
-P 10400 6950
-F 0 "#PWR016" H 10400 6950 30  0001 C CNN
-F 1 "GND" H 10400 6880 30  0001 C CNN
-F 2 "" H 10400 6950 60  0000 C CNN
-F 3 "" H 10400 6950 60  0000 C CNN
-	1    10400 6950
-	1    0    0    -1
-$EndComp
-$Comp
-L GND #PWR017
-U 1 1 5521A5BB
-P 10600 4800
-F 0 "#PWR017" H 10600 4800 30  0001 C CNN
-F 1 "GND" H 10600 4730 30  0001 C CNN
-F 2 "" H 10600 4800 60  0000 C CNN
-F 3 "" H 10600 4800 60  0000 C CNN
-	1    10600 4800
 	1    0    0    -1
 $EndComp
@@
 L PWR_FLAG #FLG035
 U 1 1 553007FD
-P 10200 4800
-F 0 "#FLG035" H 10200 4895 30  0001 C CNN
-F 1 "PWR_FLAG" H 10200 4980 30  0000 C CNN
-F 2 "" H 10200 4800 60  0000 C CNN
-F 3 "" H 10200 4800 60  0000 C CNN
-	1    10200 4800
-	1    0    0    -1
+P 9900 6900
+F 0 "#FLG035" H 9900 6995 30  0001 C CNN
+F 1 "PWR_FLAG" H 9900 7080 30  0000 C CNN
+F 2 "" H 9900 6900 60  0000 C CNN
+F 3 "" H 9900 6900 60  0000 C CNN
+	1    9900 6900
+	0    1    1    0
 $EndComp
 Text Label 6100 2150 0    60   ~ 0
@@
 	9750 6350 9750 7000
 Wire Wire Line
-	9600 6900 9750 6900
+	9600 6900 9900 6900
 Wire Wire Line
 	9600 6700 9600 6900
@@
 	9350 6450 9350 6550
 Wire Wire Line
-	10300 6750 10300 6850
-Wire Wire Line
-	10300 6850 10500 6850
-Wire Wire Line
-	10500 6850 10500 6750
-Wire Wire Line
-	10400 6850 10400 6950
-Connection ~ 10400 6850
-Wire Wire Line
-	10300 5150 10300 5050
-Wire Wire Line
-	10300 5050 10500 5050
-Wire Wire Line
-	10500 5050 10500 5150
-Wire Wire Line
-	10400 5050 10400 4700
-Wire Wire Line
-	10400 4700 10600 4700
-Wire Wire Line
-	10600 4700 10600 4800
-Connection ~ 10400 5050
-Wire Wire Line
 	9850 5550 9650 5550
 Wire Wire Line
@@
 	9850 5000 9650 5000
 Connection ~ 9650 5000
-Wire Wire Line
-	10200 4800 10200 4900
-Wire Wire Line
-	10200 4900 10400 4900
-Connection ~ 10400 4900
 Wire Wire Line
 	6000 2150 6400 2150
@@
 servo-vcc
 NoConn ~ 6000 1850
+$Comp
+L MINI-USB-B U?
+U 1 1 55B2A435
+P 10750 6050
+F 0 "U?" H 10750 5650 60  0000 C CNN
+F 1 "MINI-USB-B" H 10750 6450 60  0000 C CNN
+F 2 "" H 10750 6050 60  0000 C CNN
+F 3 "" H 10750 6050 60  0000 C CNN
+	1    10750 6050
+	1    0    0    -1
+$EndComp
+Wire Wire Line
+	9850 6550 9750 6550
+Connection ~ 9750 6550
 $EndSCHEMATC
