File: electric/scheme/cam-chassis.sch (KiCad schematic (older format))
At the start: 48 parts, among them IC1 ATMEGA8-AI, K1 pyro, P1 TST, P2 TST, P3 TST, P4 TST, P5 TST, P6 TST, P7 servo, Q3 bc857, Q4 bc847, Q5 irlml2244, Q6 NPN, Q7 irlml2244, U1 crystal-4pin, U2 MICRO-USB-B

Commit message: Replaced components to the ones I have.
Parts:
- removed U1: crystal-4pin, crystal-smd-5x3:CRYSTAL-SMD-5x3, symbol crystal-4pin
- removed U2: MICRO-USB-B, micro-usb-b:micro-usb-b, symbol MICRO-USB-B
- added U1: MINI-USB-B-4-bases, Connect:USB_Mini-B, symbol MINI-USB-B-4-bases
- added Y1: Crystal, Crystals:Crystal_HC49-U_Vertical, symbol Crystal
- C1, C2, C3, C4, C5, C6, C8: footprint Capacitors_SMD:C_0805 -> Capacitors_SMD:C_0805_HandSoldering
- C7: footprint Discret:C2V10 -> Capacitors_ThroughHole:C_Radial_D10_L13_P5
- D1, D4, D5, D6: symbol LED -> LED-RESCUE-cam-chassis
- D2, D3: symbol ZENER -> ZENER-RESCUE-cam-chassis
- R10, R11, R12, R13, R15, R16, R17, R18, R19, R20, R21, R22, R3, R5, R6, R7, R8, R9: footprint Resistors_SMD:R_0805 -> Resistors_SMD:R_0805_HandSoldering
Connections:
- no-connect marks 11 -> 9
Other:
- moved on the sheet: C2
