File: electric/scheme/_saved_cam-chassis.sch (KiCad schematic (older format))
At the start: 45 parts, among them IC1 ATMEGA8-AI, K1 pyro, P1 TST, P2 TST, P3 TST, P4 TST, P5 TST, P6 TST, P7 servo, Q3 bc857, Q4 bc847, Q5 irlml2244, Q6 NPN, Q7 irlml2244, U1 MINI-USB-B-4-bases, Y1 Crystal

Commit message: a
Changed lines of the file:
@@
 mcu-vcc
 $Comp
-L GND #PWR010
+L GND #PWR08
 U 1 1 55219BF7
 P 5000 4150
-F 0 "#PWR010" H 5000 4150 30  0001 C CNN
+F 0 "#PWR08" H 5000 4150 30  0001 C CNN
 F 1 "GND" H 5000 4080 30  0001 C CNN
 F 2 "" H 5000 4150 60  0000 C CNN
@@
 $EndComp
 $Comp
-L GND #PWR011
+L GND #PWR09
 U 1 1 5521A290
 P 9750 7000
-F 0 "#PWR011" H 9750 7000 30  0001 C CNN
+F 0 "#PWR09" H 9750 7000 30  0001 C CNN
 F 1 "GND" H 9750 6930 30  0001 C CNN
 F 2 "" H 9750 7000 60  0000 C CNN
@@
 $EndComp
 $Comp
-L GND #PWR012
+L GND #PWR010
 U 1 1 5521A361
 P 9350 6550
-F 0 "#PWR012" H 9350 6550 30  0001 C CNN
+F 0 "#PWR010" H 9350 6550 30  0001 C CNN
 F 1 "GND" H 9350 6480 30  0001 C CNN
 F 2 "" H 9350 6550 60  0000 C CNN
@@
 $EndComp
 $Comp
-L GND #PWR013
+L GND #PWR011
 U 1 1 5521A367
 P 9150 6800
-F 0 "#PWR013" H 9150 6800 30  0001 C CNN
+F 0 "#PWR011" H 9150 6800 30  0001 C CNN
 F 1 "GND" H 9150 6730 30  0001 C CNN
 F 2 "" H 9150 6800 60  0000 C CNN
@@
 $EndComp
 $Comp
-L GND #PWR014
+L GND #PWR012
 U 1 1 5521A48D
 P 10400 6950
-F 0 "#PWR014" H 10400 6950 30  0001 C CNN
+F 0 "#PWR012" H 10400 6950 30  0001 C CNN
 F 1 "GND" H 10400 6880 30  0001 C CNN
 F 2 "" H 10400 6950 60  0000 C CNN
@@
 $EndComp
 $Comp
-L GND #PWR015
+L GND #PWR013
 U 1 1 5521A5BB
 P 10600 4800
-F 0 "#PWR015" H 10600 4800 30  0001 C CNN
+F 0 "#PWR013" H 10600 4800 30  0001 C CNN
 F 1 "GND" H 10600 4730 30  0001 C CNN
 F 2 "" H 10600 4800 60  0000 C CNN
@@
 sck
 $Comp
-L VCC #PWR016
+L VCC #PWR014
 U 1 1 5521A7C3
 P 9650 4900
-F 0 "#PWR016" H 9650 5000 30  0001 C CNN
+F 0 "#PWR014" H 9650 5000 30  0001 C CNN
 F 1 "VCC" H 9650 5000 30  0000 C CNN
 F 2 "" H 9650 4900 60  0000 C CNN
@@
 $EndComp
 $Comp
-L GND #PWR017
+L GND #PWR015
 U 1 1 5521B56E
 P 3150 7650
-F 0 "#PWR017" H 3150 7650 30  0001 C CNN
+F 0 "#PWR015" H 3150 7650 30  0001 C CNN
 F 1 "GND" H 3150 7580 30  0001 C CNN
 F 2 "" H 3150 7650 60  0000 C CNN
@@
 $EndComp
 $Comp
-L VCC #PWR018
+L VCC #PWR016
 U 1 1 5521BB76
 P 700 5200
-F 0 "#PWR018" H 700 5300 30  0001 C CNN
+F 0 "#PWR016" H 700 5300 30  0001 C CNN
 F 1 "VCC" H 700 5300 30  0000 C CNN
 F 2 "" H 700 5200 60  0000 C CNN
@@
 $EndComp
 $Comp
-L VCC #PWR019
+L VCC #PWR017
 U 1 1 5521C271
-P 7650 5900
-F 0 "#PWR019" H 7650 6000 30  0001 C CNN
-F 1 "VCC" H 7650 6000 30  0000 C CNN
-F 2 "" H 7650 5900 60  0000 C CNN
-F 3 "" H 7650 5900 60  0000 C CNN
-	1    7650 5900
-	1    0    0    -1
-$EndComp
-$Comp
-L GND #PWR020
+P 10900 3950
+F 0 "#PWR017" H 10900 4050 30  0001 C CNN
+F 1 "VCC" H 10900 4050 30  0000 C CNN
+F 2 "" H 10900 3950 60  0000 C CNN
+F 3 "" H 10900 3950 60  0000 C CNN
+	1    10900 3950
+	1    0    0    -1
+$EndComp
+$Comp
+L GND #PWR018
 U 1 1 5521C30D
 P 7650 6500
-F 0 "#PWR020" H 7650 6500 30  0001 C CNN
+F 0 "#PWR018" H 7650 6500 30  0001 C CNN
 F 1 "GND" H 7650 6430 30  0001 C CNN
 F 2 "" H 7650 6500 60  0000 C CNN
@@
 $EndComp
 $Comp
-L GND #PWR021
+L GND #PWR019
 U 1 1 5524036E
 P 3650 6050
-F 0 "#PWR021" H 3650 6050 30  0001 C CNN
+F 0 "#PWR019" H 3650 6050 30  0001 C CNN
 F 1 "GND" H 3650 5980 30  0001 C CNN
 F 2 "" H 3650 6050 60  0000 C CNN
@@
 $EndComp
 $Comp
-L GND #PWR022
+L GND #PWR020
 U 1 1 552406B4
 P 6750 5550
-F 0 "#PWR022" H 6750 5550 30  0001 C CNN
+F 0 "#PWR020" H 6750 5550 30  0001 C CNN
 F 1 "GND" H 6750 5480 30  0001 C CNN
 F 2 "" H 6750 5550 60  0000 C CNN
@@
 $EndComp
 $Comp
-L GND #PWR023
+L GND #PWR021
 U 1 1 55240AD0
 P 10350 4400
-F 0 "#PWR023" H 10350 4400 30  0001 C CNN
+F 0 "#PWR021" H 10350 4400 30  0001 C CNN
 F 1 "GND" H 10350 4330 30  0001 C CNN
 F 2 "" H 10350 4400 60  0000 C CNN
@@
 $EndComp
 $Comp
-L GND #PWR024
+L GND #PWR022
 U 1 1 55240C73
 P 10650 4400
-F 0 "#PWR024" H 10650 4400 30  0001 C CNN
+F 0 "#PWR022" H 10650 4400 30  0001 C CNN
 F 1 "GND" H 10650 4330 30  0001 C CNN
 F 2 "" H 10650 4400 60  0000 C CNN
@@
 $EndComp
 $Comp
-L GND #PWR025
+L GND #PWR023
 U 1 1 55240C87
 P 10950 4400
-F 0 "#PWR025" H 10950 4400 30  0001 C CNN
+F 0 "#PWR023" H 10950 4400 30  0001 C CNN
 F 1 "GND" H 10950 4330 30  0001 C CNN
 F 2 "" H 10950 4400 60  0000 C CNN
@@
 $EndComp
 $Comp
-L GND #PWR026
+L GND #PWR024
 U 1 1 55241757
 P 9000 3500
-F 0 "#PWR026" H 9000 3500 30  0001 C CNN
+F 0 "#PWR024" H 9000 3500 30  0001 C CNN
 F 1 "GND" H 9000 3430 30  0001 C CNN
 F 2 "" H 9000 3500 60  0000 C CNN
@@
 $EndComp
 $Comp
-L GND #PWR027
+L GND #PWR025
 U 1 1 552419C1
 P 9600 3500
-F 0 "#PWR027" H 9600 3500 30  0001 C CNN
+F 0 "#PWR025" H 9600 3500 30  0001 C CNN
 F 1 "GND" H 9600 3430 30  0001 C CNN
 F 2 "" H 9600 3500 60  0000 C CNN
@@
 $EndComp
 $Comp
-L GND #PWR028
+L GND #PWR026
 U 1 1 552FF855
 P 7800 2250
-F 0 "#PWR028" H 7800 2250 30  0001 C CNN
+F 0 "#PWR026" H 7800 2250 30  0001 C CNN
 F 1 "GND" H 7800 2180 30  0001 C CNN
 F 2 "" H 7800 2250 60  0000 C CNN
@@
 pyro-sen
 $Comp
-L VCC #PWR029
+L VCC #PWR027
 U 1 1 552FF5E1
 P 7650 1750
-F 0 "#PWR029" H 7650 1850 30  0001 C CNN
+F 0 "#PWR027" H 7650 1850 30  0001 C CNN
 F 1 "VCC" H 7650 1850 30  0000 C CNN
 F 2 "" H 7650 1750 60  0000 C CNN
@@
 $EndComp
 $Comp
-L VCC #PWR030
+L VCC #PWR028
 U 1 1 5530007B
 P 7100 4050
-F 0 "#PWR030" H 7100 4150 30  0001 C CNN
+F 0 "#PWR028" H 7100 4150 30  0001 C CNN
 F 1 "VCC" H 7100 4150 30  0000 C CNN
 F 2 "" H 7100 4050 60  0000 C CNN
@@
 $EndComp
 $Comp
-L GND #PWR031
+L GND #PWR029
 U 1 1 55300137
 P 7400 4100
-F 0 "#PWR031" H 7400 4100 30  0001 C CNN
+F 0 "#PWR029" H 7400 4100 30  0001 C CNN
 F 1 "GND" H 7400 4030 30  0001 C CNN
 F 2 "" H 7400 4100 60  0000 C CNN
@@
 mosi
 $Comp
-L PWR_FLAG #FLG032
+L PWR_FLAG #FLG030
 U 1 1 5530026F
 P 3650 5100
-F 0 "#FLG032" H 3650 5195 30  0001 C CNN
+F 0 "#FLG030" H 3650 5195 30  0001 C CNN
 F 1 "PWR_FLAG" H 3650 5280 30  0000 C CNN
 F 2 "" H 3650 5100 60  0000 C CNN
@@
 $EndComp
 $Comp
-L PWR_FLAG #FLG033
+L PWR_FLAG #FLG031
 U 1 1 553007FD
 P 10200 4800
-F 0 "#FLG033" H 10200 4895 30  0001 C CNN
+F 0 "#FLG031" H 10200 4895 30  0001 C CNN
 F 1 "PWR_FLAG" H 10200 4980 30  0000 C CNN
 F 2 "" H 10200 4800 60  0000 C CNN
@@
 NoConn ~ 6000 1350
 $Comp
-L VCC #PWR034
+L VCC #PWR032
 U 1 1 55300EC2
 P 9600 1450
-F 0 "#PWR034" H 9600 1550 30  0001 C CNN
+F 0 "#PWR032" H 9600 1550 30  0001 C CNN
 F 1 "VCC" H 9600 1550 30  0000 C CNN
 F 2 "" H 9600 1450 60  0000 C CNN
@@
 $EndComp
 $Comp
-L VCC #PWR035
+L VCC #PWR033
 U 1 1 55300EC8
 P 10350 1950
-F 0 "#PWR035" H 10350 2050 30  0001 C CNN
+F 0 "#PWR033" H 10350 2050 30  0001 C CNN
 F 1 "VCC" H 10350 2050 30  0000 C CNN
 F 2 "" H 10350 1950 60  0000 C CNN
@@
 $EndComp
 $Comp
-L PWR_FLAG #FLG036
+L PWR_FLAG #FLG034
 U 1 1 552FFAA1
 P 9850 4900
-F 0 "#FLG036" H 9850 4995 30  0001 C CNN
+F 0 "#FLG034" H 9850 4995 30  0001 C CNN
 F 1 "PWR_FLAG" H 9850 5080 30  0000 C CNN
 F 2 "" H 9850 4900 60  0000 C CNN
